Commit message: burger box

File: assets/urdf/soomac_description/urdf/burgerbox.urdf (robot description, URDF)
Before this commit: robot basket, 1 links, 0 joints
Links:
- link base_link: geometry collision mesh filename=package://soomac_description/meshes/burger_box/files/BOTTOM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 scale=0.003 0.003 0.003; visual mesh filename=package://soomac_description/meshes/burger_box/files/BOTTOM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 scale=0.003 0.003 0.003
