Commit message: soomac origin change version

File: assets/urdf/soomac_description/urdf/soomac.urdf (robot description, URDF)
Before this commit: robot soomac, 8 links, 7 joints
Joints:
- joint link2_to_base_link: limit (none) -> lower=-6.28318 upper=6.28318 effort=330.0 velocity=2.0944
- joint link3_to_link2: limit (none) -> lower=-6.28318 upper=6.28318 effort=330.0 velocity=2.0944
- joint link4_to_link3: limit (none) -> lower=-6.28318 upper=6.28318 effort=330.0 velocity=2.0944
- joint link5_to_link4: limit (none) -> lower=-6.28318 upper=6.28318 effort=330.0 velocity=2.0944
- joint link6_to_link5: limit (none) -> lower=-6.28318 upper=6.28318 effort=330.0 velocity=2.0944
- joint link7_to_link6: origin xyz=0.23447 -0.073579 0.345 rpy=0 0 0 -> xyz=-0.0205 0.0485 0.0 rpy=0 0 0
- joint link8_to_link6: limit lower=0.0 upper=0.0281 effort=100 velocity=100 -> lower=0.00295 upper=0.031 effort=100 velocity=100; origin xyz=0.28842 -0.073579 0.345 rpy=0 0 0 -> xyz=-0.0205 0.0485 0.0 rpy=0 0 0

Commit message: soomac pnp prac

File: assets/urdf/soomac_description/urdf/soomac.urdf (robot description, URDF)
Before this commit: robot (soomac, 8 links, 7 joints
Joints:
- joint Slider 8: child link8_finger_l_1 -> link7_finger_r_1; limit lower=0.003 upper=0.031 effort=100 velocity=100 -> lower=-0.031 upper=0.000 effort=100 velocity=100; origin xyz=-0.0205 0.0485 0.0 rpy=0 0 0 -> xyz=0.0 0.05 0.0 rpy=0 0 0
- joint Slider 9: child link7_finger_r_1 -> link8_finger_l_1; limit lower=-0.031 upper=-0.003 effort=100 velocity=100 -> lower=0.000 upper=0.031 effort=100 velocity=100; origin xyz=-0.0205 0.0485 0.0 rpy=0 0 0 -> xyz=0.0 0.05 0.0 rpy=0 0 0

Commit message: orientation error control

File: assets/urdf/soomac_description/urdf/soomac.urdf (robot description, URDF)
Before this commit: robot (soomac, 8 links, 7 joints
Links:
- added link grip_site; visual sphere radius=0.005
Joints:
- added joint grip_joint: type fixed, parent link6_gripper_1, child grip_site, origin xyz=0 0.1 0 rpy=1.57079632679 0 0
