Commit message: soomac_description edit

File: assets/urdf/soomac_description_0/urdf/materials.xacro (robot description, xacro)
@@ -1,4 +1,4 @@
 <?xml version="1.0" ?>
-<robot name="(Unsaved)" xmlns:xacro="http://www.ros.org/wiki/xacro" >
+<robot name="soomac" xmlns:xacro="http://www.ros.org/wiki/xacro" >
 <material name="silver">
   <color rgba="0.700 0.700 0.700 1.000"/>

File: assets/urdf/soomac_description_0/urdf/soomac.urdf (robot description, URDF)
Before this commit: robot (soomac, 8 links, 7 joints
Links:
- link base_link: mass 0.31335946697273154 -> 1.5026706265949556
- link link2_1: mass 0.3584319251227706 -> 1.718809170564294
- link link3_1: mass 0.22806001266597076 -> 1.0936292604935065
- link link4_1: mass 0.21493203724961896 -> 1.030675926945332
- link link5_1: mass 0.11465885199939559 -> 0.549830169942123
- link link6_gripper_1: mass 0.13960741404599217 -> 0.6694674405992905
- link link7_finger_r_1: mass 0.04558518327790625 -> 0.2185972441854391
- link link8_finger_l_1: mass 0.04558023056880734 -> 0.21857349417540464
Joints:
- removed joint Slider 8
- removed joint Slider 9
- added joint link7_to_link6: type prismatic, parent link6_gripper_1, child link7_finger_r_1, origin xyz=-0.0205 0.0485 0.0 rpy=0 0 0, axis -1.0 -0.0 0.0, limit lower=0.0 upper=0.0281 effort=100 velocity=100
- added joint link8_to_link6: type prismatic, parent link6_gripper_1, child link8_finger_l_1, origin xyz=-0.0205 0.0485 0.0 rpy=0 0 0, axis 1.0 -0.0 0.0, limit lower=0.00295 upper=0.031 effort=100 velocity=100
- joint link2_to_base_link: limit (none) -> lower=-6.28318 upper=6.28318 effort=330.0 velocity=2.0944
- joint link3_to_link2: limit (none) -> lower=-6.28318 upper=6.28318 effort=330.0 velocity=2.0944
- joint link4_to_link3: limit (none) -> lower=-6.28318 upper=6.28318 effort=330.0 velocity=2.0944; origin xyz=0.040375 -0.000745 0.303249 rpy=0 0 0 -> xyz=0.040375 0.0 0.30325 rpy=0 0 0
- joint link5_to_link4: limit (none) -> lower=-6.28318 upper=6.28318 effort=330.0 velocity=2.0944; origin xyz=-0.03975 0.327749 0.000656 rpy=0 0 0 -> xyz=-0.03975 0.32775 -1.3e-05 rpy=0 0 0
- joint link6_to_link5: axis -0.0 1.0 0.0 -> 0.0 1.0 0.0; limit (none) -> lower=-6.28318 upper=6.28318 effort=330.0 velocity=2.0944
